Commit message: adding readme and table scene. Next TODO: adding camera

File: src/lerobot_description/urdf/so101_base.xacro (robot description, xacro)
@@ -6,5 +6,4 @@
 -->
 <robot xmlns:xacro="http://www.ros.org/wiki/xacro">
-	<!-- Links -->
 	<link name="world" />
 	<joint name="base_joint" type="fixed">
@@ -20,5 +19,5 @@
 		<color rgba="0.1 0.1 0.1 1.0" />
 	</material>
-	<!-- Link base -->
+	<!-- Link base. Note that original file had z origin offsets here which I removed to make the bottom of the base link align with the bottom of the part -->
 	<link name="base">
 		<inertial>
@@ -30,5 +29,5 @@
 		<!-- Part base_motor_holder_so101_v1 -->
 		<visual>
-			<origin xyz="0.0206915 0.0221255 0.0300817" rpy="1.5708 -1.23909e-16 2.33147e-15" />
+			<origin xyz="0.0206915 0.0221255 0.0" rpy="1.5708 -1.23909e-16 2.33147e-15" />
 			<geometry>
 				<mesh
@@ -38,5 +37,5 @@
 		</visual>
 		<collision>
-			<origin xyz="0.0206915 0.0221255 0.0300817" rpy="1.5708 -1.23909e-16 2.33147e-15" />
+			<origin xyz="0.0206915 0.0221255 0.0" rpy="1.5708 -1.23909e-16 2.33147e-15" />
 			<geometry>
 				<mesh
@@ -46,5 +45,5 @@
 		<!-- Part base_so101_v2 -->
 		<visual>
-			<origin xyz="0.0207909 0.0221255 0.0300817" rpy="1.5708 -0 0" />
+			<origin xyz="0.0207909 0.0221255 0.0" rpy="1.5708 -0 0" />
 			<geometry>
 				<mesh filename="package://lerobot_description/meshes/so101/base_so101_v2.stl" />
@@ -53,5 +52,5 @@
 		</visual>
 		<collision>
-			<origin xyz="0.0207909 0.0221255 0.0300817" rpy="1.5708 -0 0" />
+			<origin xyz="0.0207909 0.0221255 0.0" rpy="1.5708 -0 0" />
 			<geometry>
 				<mesh filename="package://lerobot_description/meshes/so101/base_so101_v2.stl" />
@@ -74,5 +73,5 @@
 		<!-- Part waveshare_mounting_plate_so101_v2 -->
 		<visual>
-			<origin xyz="0.0205915 0.0467435 0.0798817" rpy="1.5708 -1.21716e-14 2.33147e-15" />
+			<origin xyz="0.0205915 0.0467435 0.0498" rpy="1.5708 -1.21716e-14 2.33147e-15" />
 			<geometry>
 				<mesh
@@ -82,5 +81,5 @@
 		</visual>
 		<collision>
-			<origin xyz="0.0205915 0.0467435 0.0798817" rpy="1.5708 -1.21716e-14 2.33147e-15" />
+			<origin xyz="0.0205915 0.0467435 0.0498" rpy="1.5708 -1.21716e-14 2.33147e-15" />
 			<geometry>
 				<mesh

Commit message: adding realsense camera to gazebo and URDF. Next TODO: rename things to fit what I am actually doing

File: src/lerobot_description/urdf/so101_base.xacro (robot description, xacro)
@@ -6,5 +6,4 @@
 -->
 <robot xmlns:xacro="http://www.ros.org/wiki/xacro">
-	<link name="world" />
 	<joint name="base_joint" type="fixed">
 		<parent link="world" />

File: src/lerobot_description/urdf/so101_ros2_control.xacro (robot description, xacro)
@@ -3,6 +3,9 @@
     <ros2_control name="RobotSystem" type="system">
         <!-- ros2_control Gazebo -->
+        <!-- Note, for real hardware need to add different plugin to expose the hardware interfaces -->
         <hardware>
-            <plugin>gz_ros2_control/GazeboSimSystem</plugin>
+            <xacro:if value="$(arg use_sim)">
+                <plugin>gz_ros2_control/GazeboSimSystem</plugin>
+            </xacro:if>
         </hardware>
         <joint name="1">
